Commit message: Automatic grabbing within proximity works

File: controllers/grocery_shopper/robot_urdf.urdf (robot description, URDF)
Before this commit: robot TIAGo Steel, 52 links, 51 joints
Links:
- added link rgb_camera_optical_frame
Joints:
- added joint head_2_rgb_camera_joint: type fixed, parent head_2_link, child rgb_camera_optical_frame, origin xyz=-0.01177 0.0800 -0.025 rpy=0 -1.5708 3.14159
